Commit message: Added stl files and fixed setup.py.

File: ros2_ws/src/robot_consepts_viz_pkg/urdf/h_bot.urdf (robot description, URDF)
Before this commit: robot h_bot, 1 links, 0 joints
Links:
- link base_link: geometry visual mesh filename=package://robot_consepts_viz_pkg/meshes/stl/base.stl

Commit message: Switched back to .dae files for visual geometry.

File: ros2_ws/src/robot_consepts_viz_pkg/urdf/h_bot.urdf (robot description, URDF)
Before this commit: robot h_bot, 1 links, 0 joints
Links:
- link base_link: geometry visual mesh filename=package://robot_consepts_viz_pkg/meshes/dae/base.dae

Commit message: Adding link_1 and joint_1 to h_bot.

File: ros2_ws/src/robot_consepts_viz_pkg/urdf/h_bot.urdf (robot description, URDF)
Before this commit: robot h_bot, 1 links, 0 joints
Links:
- added link link_1; visual mesh filename=package://robot_consepts_viz_pkg/meshes/dae/joint1.dae
Joints:
- added joint joint_1: type continuous, parent base_link, child link_1

Commit message: Switching from continuous joint to revolute.

File: ros2_ws/src/robot_consepts_viz_pkg/urdf/h_bot.urdf (robot description, URDF)
Before this commit: robot h_bot, 2 links, 1 joints
Joints:
- joint joint_1: limit (none) -> lower=${-pi} upper=${pi} effort=1000.0 velocity=0.5; type continuous -> revolute

Commit message: Changing originand axis of rotation for joint 1.

File: ros2_ws/src/robot_consepts_viz_pkg/urdf/h_bot.urdf (robot description, URDF)
Before this commit: robot h_bot, 2 links, 1 joints
Joints:
- joint joint_1: axis (none) -> 0 0 1; origin (none) -> xyz=0 0 0.1425 rpy=0 0 0

Commit message: Adding link_2 and joint_2.

File: ros2_ws/src/robot_consepts_viz_pkg/urdf/h_bot.urdf (robot description, URDF)
Before this commit: robot h_bot, 2 links, 1 joints
Links:
- added link link_2; visual mesh filename=package://robot_consepts_viz_pkg/meshes/dae/joint2.dae
Joints:
- added joint joint_2: type revolute, parent link_1, child link_2, origin xyz=0 0 0.1425 rpy=${-pi/2} ${pi/2} 0, axis 0 0 1, limit lower=${-pi} upper=${pi} effort=1000.0 velocity=0.5

Commit message: Adding link_3 and joint_3.

File: ros2_ws/src/robot_consepts_viz_pkg/urdf/h_bot.urdf (robot description, URDF)
Before this commit: robot h_bot, 3 links, 2 joints
Links:
- added link link_3; visual mesh filename=package://robot_consepts_viz_pkg/meshes/dae/joint3.dae
Joints:
- added joint joint_3: type revolute, parent link_2, child link_3, origin xyz=-0.7 0 0 rpy=${pi/2} ${pi} 0, axis 0 1 0, limit lower=${-pi} upper=${pi} effort=1000.0 velocity=0.5

Commit message: Adding link_4 and joint_4.

File: ros2_ws/src/robot_consepts_viz_pkg/urdf/h_bot.urdf (robot description, URDF)
Before this commit: robot h_bot, 4 links, 3 joints
Links:
- added link link_4; visual mesh filename=package://robot_consepts_viz_pkg/meshes/dae/joint4.dae
Joints:
- added joint joint_4: type revolute, parent link_3, child link_4, origin xyz=0 0 0.65 rpy=${pi/2} 0 0, axis 0 1 0, limit lower=${-pi} upper=${pi} effort=1000.0 velocity=0.5

Commit message: Adding link_5 and joint_5.

File: ros2_ws/src/robot_consepts_viz_pkg/urdf/h_bot.urdf (robot description, URDF)
Before this commit: robot h_bot, 5 links, 4 joints
Links:
- added link link_5; visual mesh filename=package://robot_consepts_viz_pkg/meshes/dae/joint5.dae
Joints:
- added joint joint_5: type revolute, parent link_4, child link_5, origin xyz=0 0 0 rpy=${-pi/2} 0 0, axis 0 1 0, limit lower=${-pi} upper=${pi} effort=1000.0 velocity=0.5

Commit message: Adding link_6 and joint_6.

File: ros2_ws/src/robot_consepts_viz_pkg/urdf/h_bot.urdf (robot description, URDF)
Before this commit: robot h_bot, 6 links, 5 joints
Links:
- added link link_6; visual mesh filename=package://robot_consepts_viz_pkg/meshes/dae/joint6.dae
Joints:
- added joint joint_6: type revolute, parent link_5, child link_6, origin xyz=0 0 0.17 rpy=0 0 0, axis 0 0 1, limit lower=${-pi} upper=${pi} effort=1000.0 velocity=0.5

Commit message: Joint frames match exercise more closely.

File: ros2_ws/src/robot_consepts_viz_pkg/urdf/h_bot.urdf (robot description, URDF)
Before this commit: robot h_bot, 7 links, 6 joints
Joints:
- joint joint_1: origin xyz=0 0 0.1425 rpy=0 0 0 -> xyz=0 0 0 rpy=0 0 0
- joint joint_2: origin xyz=0 0 0.1425 rpy=${-pi/2} ${pi/2} 0 -> xyz=0 0 0.285 rpy=${-pi/2} 0 0
- joint joint_3: axis 0 1 0 -> 0 0 1; origin xyz=-0.7 0 0 rpy=${pi/2} ${pi} 0 -> xyz=0 -0.7 0 rpy=0 0 ${-pi/2}
- joint joint_4: axis 0 1 0 -> 0 0 1; origin xyz=0 0 0.65 rpy=${pi/2} 0 0 -> xyz=0 0 0 rpy=${-pi/2} 0 0
- joint joint_5: axis 0 1 0 -> 0 0 1; origin xyz=0 0 0 rpy=${-pi/2} 0 0 -> xyz=0 0 0.65 rpy=${pi/2} 0 0
- joint joint_6: origin xyz=0 0 0.17 rpy=0 0 0 -> xyz=0 0 0 rpy=${-pi/2} 0 0
